File: WS2812Controller.kicad_pcb (KiCad board)
At the start: 2 copper layers, 49.4 x 32.3 mm, 19 parts, among them J1 USB_B_Micro, J2 Conn_01x05_Male, J3 Conn_01x03, J4 Conn_01x02_Male, SW1 SW_Reset, SW2 SW_GPIO0, U1 AMS1117-3.3, U2 ESP-12F

Commit message: v0.3
Parts:
- removed J4: Conn_01x02_Male, TerminalBlock:TerminalBlock_bornier-2_P5.08mm
- removed the REF** at (155.9, 98.6)
- added F1: Fuse, halibs:Fuse-PTF75_Stelvio, F.Cu at (135.9, 105.5)
- added REF**: MountingHole_3.2mm_M3, MountingHole:MountingHole_3.2mm_M3, F.Cu at (156.7, 102.6)
- added REF**: MountingHole_3.2mm_M3, MountingHole:MountingHole_3.2mm_M3, F.Cu at (114.2, 73.8)
- J1: value USB_B_Micro -> Conn_01x04_Male; footprint Connector_USB:USB_Micro-B_Molex_47346-0001 -> TerminalBlock_Phoenix:TerminalBlock_Phoenix_MPT-0,5-4-2.54_1x04_P2.54mm_Horizontal
- moved R4 20.0 mm to (150.1, 97.9), turned to 270 degrees
- moved J1 6.13 mm to (114.6, 81.6)
- moved G*** 1.67 mm to (137.0, 88.4)
Connections:
- J1 pad 1: +5V -> /SUPPLY
- J1 pad 2: Net-(J1-Pad2) -> /SUPPLY
- J1 pad 3: Net-(J1-Pad3) -> GND
- J1 pad 4: Net-(J1-Pad4) -> GND
Routing:
- net /SUPPLY: track 0.00 -> 36.7 mm
- net Net-(J1-Pad6): track 10.8 -> 0.00 mm
- net +3V3: track 73.9 -> 81.5 mm
- net Net-(R4-Pad2): track 18.2 -> 13.7 mm
- net +5V: track 80.0 -> 76.1 mm
- net GND: track 2.95 -> 0.00 mm, vias 1 -> 0
- net Net-(J3-Pad2): track 7.44 -> 8.10 mm
Other:
- board size 49.4 x 32.3 mm -> 49.4 x 35.8 mm
- net class 5V removed
- net class Closer removed
- net class Fet added: clearance 0.3, trace_width 0.5, via_dia 0.8, via_drill 0.4
- board text added: "+5V"
- board text added: "v0.3 2021/05/12"
- board text removed: "+"
- board text removed: "-"
- board text removed: "AMS1117-3.3"
- board text removed: "v0.2 2021/05/07"

Commit message: Readme
Parts:
- C1, C2: value 100µF -> 100nF
Other:
- board text added: "v0.4 2021/06/10"
- board text removed: "v0.3 2021/05/12"

Commit message: Bigger tracks for 5V supply
Routing:
- net /SUPPLY: track 36.7 -> 75.2 mm
- net +5V: track 76.1 -> 107.7 mm
- net GND: vias 0 -> 1
Other:
- net class Fet: trace_width 0.5 -> 1.5
- board text added: "v0.4 2021/06/21"
- board text removed: "v0.4 2021/06/10"

Commit message: v0.4
Parts:
- removed the G*** at (137.0, 88.4)
- added G***: LOGO, halibs:Logo, B.Cu at (149.1, 94.0)
- added U3: SN74AHCT125, halibs:SN74AHCT125D, B.Cu at (136.6, 81.5)
Connections:
- J1 pad 1: /SUPPLY -> GND
- J1 pad 2: /SUPPLY -> GND
- J1 pad 3: GND -> /SUPPLY
- J1 pad 4: GND -> /SUPPLY
- R6 pad 2: GPIO4 -> DATA
Routing:
- net +5V: track 107.7 -> 166.3 mm
- net DATA: track 0.00 -> 13.2 mm, vias 0 -> 1
- net /SUPPLY: track 75.2 -> 64.2 mm
- net GPIO4: track 8.00 -> 4.81 mm, vias 0 -> 1
Other:
- board text added: "5A max."
- board text added: "v0.4 2021/09/29"
- board text removed: "v0.4 2021/06/21"

Commit message: v0.5
Parts:
- removed the G*** at (149.1, 94.0)
- added G***: LOGO, halibs:Logo_20mm, B.Cu at (136.4, 88.0)
- added REF**: WEEE-Logo_4.2x6mm_SilkScreen, Symbol:WEEE-Logo_4.2x6mm_SilkScreen, F.Cu at (115.2, 79.4)
- U3: moved to F.Cu
- moved J3 39.3 mm to (115.8, 83.9), turned to 270 degrees
- moved R1 34.6 mm to (155.3, 73.7), turned to 270 degrees
- moved R3 30.0 mm to (155.3, 77.7), turned to 270 degrees
- moved C2 29.6 mm to (143.7, 73.7), turned to 90 degrees
- moved J2 29.1 mm to (150.9, 102.6), turned to 270 degrees
- moved U1 28.7 mm to (149.7, 75.6), turned to 0 degrees
- moved C1 24.2 mm to (143.7, 77.5), turned to 270 degrees
- moved R6 24.1 mm to (129.7, 75.2)
- moved SW2 19.4 mm to (132.1, 95.0), turned to 90 degrees
- moved C3 19.4 mm to (122.5, 77.5), turned to 90 degrees
- moved R5 16.9 mm to (137.7, 102.0)
- moved R2 16.9 mm to (133.3, 102.0)
- moved R4 15.1 mm to (135.5, 102.0), turned to 90 degrees
- moved F1 14.1 mm to (129.2, 93.1), turned to 270 degrees
- moved U2 13.3 mm to (148.0, 89.5), turned to 270 degrees
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Routing:
- net +5V: track 166.3 -> 66.8 mm, vias 0 -> 1
- net /SUPPLY: track 64.2 -> 22.8 mm
- net GPIO4: track 4.81 -> 34.0 mm, vias 1 -> 2
- net /RST: track 7.83 -> 32.3 mm, vias 0 -> 2
- net +3V3: track 81.5 -> 57.7 mm
- net Net-(J3-Pad2): track 8.10 -> 28.6 mm
- net GND: track 0.10 -> 16.1 mm, vias 1 -> 2
- net /EN: track 6.84 -> 13.8 mm
- net Net-(R2-Pad1): track 2.62 -> 8.66 mm
- net RX: track 3.51 -> 9.39 mm
- net Net-(R4-Pad2): track 13.7 -> 8.50 mm
- net TX: track 3.46 -> 8.17 mm
- net GPIO0: track 22.2 -> 26.5 mm, vias 0 -> 3
- net DATA: track 13.2 -> 9.70 mm, vias 1 -> 0
Other:
- outline, holes or cut-outs redrawn
- net class Fet: trace_width 1.5 -> 0.25
- board text added: "v0.5"
- board text removed: "+5V"
- board text removed: "10kΩ"
- board text removed: "330Ω"
- board text removed: "v0.4 2021/09/29"

Commit message: Fixed minor connection issues
Parts:
- U3: footprint halibs:SN74AHCT125D -> haus-automatisierung:SN74AHCT125D
Connections:
- U2 pad 10: Net-(U2-Pad10) -> unconnected-(U2-Pad10)
- U2 pad 11: Net-(U2-Pad11) -> unconnected-(U2-Pad11)
- U2 pad 12: Net-(U2-Pad12) -> unconnected-(U2-Pad12)
- U2 pad 13: Net-(U2-Pad13) -> unconnected-(U2-Pad13)
- U2 pad 14: Net-(U2-Pad14) -> unconnected-(U2-Pad14)
- U2 pad 2: Net-(U2-Pad2) -> unconnected-(U2-Pad2)
- U2 pad 20: Net-(U2-Pad20) -> unconnected-(U2-Pad20)
- U2 pad 4: Net-(U2-Pad4) -> unconnected-(U2-Pad4)
- U2 pad 5: Net-(U2-Pad5) -> unconnected-(U2-Pad5)
- U2 pad 6: Net-(U2-Pad6) -> unconnected-(U2-Pad6)
- U2 pad 7: Net-(U2-Pad7) -> unconnected-(U2-Pad7)
- U2 pad 9: Net-(U2-Pad9) -> unconnected-(U2-Pad9)
- U3 pad 11: Net-(U3-Pad11) -> unconnected-(U3-Pad11)
- U3 pad 12: Net-(U3-Pad12) -> unconnected-(U3-Pad12)
- U3 pad 5: Net-(U3-Pad5) -> unconnected-(U3-Pad5)
- U3 pad 6: Net-(U3-Pad6) -> unconnected-(U3-Pad6)
- U3 pad 8: Net-(U3-Pad8) -> unconnected-(U3-Pad8)
- U3 pad 9: Net-(U3-Pad9) -> unconnected-(U3-Pad9)
Routing:
- net +5V: track 66.8 -> 66.1 mm
- net /RST: track 32.3 -> 31.7 mm
- net GPIO0: track 26.5 -> 25.9 mm
Other:
- net class Default removed
- net class Fet removed
- board text added: "v0.6"
- board text removed: "v0.5"
