File: WS2812Controller.kicad_pcb (KiCad board)
At the start: 2 copper layers, 49.4 x 35.8 mm, 22 parts, among them J1 Conn_01x04_Male, J2 Conn_01x05_Male, J3 Conn_01x03, SW1 SW_Reset, SW2 SW_GPIO0, U1 AMS1117-3.3, U2 ESP-12F, U3 SN74AHCT125

Commit message: v0.7
Parts:
- removed the G*** at (136.4, 88.0)
- added G***: LOGO, haus-automatisierung:Logo2024, B.Cu at (145.1, 89.7)
Other:
- board text added: "v0.7"
- board text removed: "v0.6"

Commit message: Update
Routing:
- net GND: track 16.1 -> 11.9 mm
Other:
- board text added: "v0.8"
- board text removed: "v0.7"
Changed lines of the file:
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@@
 		(title "WS2812 Controller")
 		(date "2024-05-07")
-		(rev "0.7")
+		(rev "0.8")
 		(company "haus-automatisierung.com")
 		(comment 1 "Matthias Kleine")
@@
 		)
 	)
-	(gr_text "v0.7"
+	(gr_text "v0.8"
 		(at 115.7224 104.267 0)
 		(layer "F.SilkS")
@@
 	)
 	(segment
-		(start 134.652 78.3356)
-		(end 134.652 79.3356)
-		(width 0.25)
-		(layer "F.Cu")
-		(net 2)
-	)
-	(segment
 		(start 145.93014 72.70104)
 		(end 146.56014 73.33104)
@@
 		(width 0.25)
 		(layer "F.Cu")
-		(net 2)
-	)
-	(segment
-		(start 134.652 79.3356)
-		(end 133.04906 80.93854)
-		(width 0.25)
-		(layer "F.Cu")
-		(net 2)
-	)
-	(segment
-		(start 133.04906 80.93854)
-		(end 132.14096 80.93854)
-		(width 0.25)
-		(layer "F.Cu")
