File: WS2812Controller.sch (KiCad schematic (older format))
At the start: 17 parts, among them J1 USB_B_Micro, J2 Conn_01x05_Male, J3 Conn_01x03, J4 Conn_01x02_Male, SW1 SW_Reset, SW2 SW_GPIO0, U1 AMS1117-3.3, U2 ESP-12F

Commit message: v0.3
Parts:
- removed J1: USB_B_Micro, Connector_USB:USB_Micro-B_Molex_47346-0001, symbol WS2812Controller-rescue:USB_B_Micro-Connector
- removed J4: Conn_01x02_Male, TerminalBlock:TerminalBlock_bornier-2_P5.08mm, symbol Connector:Conn_01x02_Male
- added F1: Fuse, halibs:Fuse-PTF75_Stelvio, symbol Device:Fuse
- added J1: Conn_01x04_Male, TerminalBlock_Phoenix:TerminalBlock_Phoenix_MPT-0,5-4-2.54_1x04_P2.54mm_Horizontal, symbol Connector:Conn_01x04_Male
Connections:
- net +5V: now also F1.1
- net GND: now also J1.3 (Pin_3), J1.4 (Pin_4)
- new net SUPPLY: F1.2, J1.1 (Pin_1), J1.2 (Pin_2)
- no-connect marks 16 -> 12
Changed lines of the file:
@@
 Sheet 1 1
 Title "WS2812 Controller"
-Date "2021-05-07"
-Rev "0.2"
+Date "2021-05-12"
+Rev "0.3"
 Comp "haus-automatisierung.com"
 Comment1 "Matthias Kleine"
@@
 $EndComp
 Connection ~ 7100 3400
-$Comp
-L WS2812Controller-rescue:USB_B_Micro-Connector J1
-U 1 1 5C938411
-P 1600 1900
-F 0 "J1" V 1350 2100 50  0000 L CNN
-F 1 "USB_B_Micro" V 1350 1600 50  0000 L CNN
-F 2 "Connector_USB:USB_Micro-B_Molex_47346-0001" H 1750 1850 50  0001 C CNN
-F 3 "~" H 1750 1850 50  0001 C CNN
-	1    1600 1900
-	0    -1   -1   0
-$EndComp
-Wire Wire Line
-	2000 1900 2150 1900
 Connection ~ 2700 1900
 $Comp
@@
 NoConn ~ 6500 2500
 NoConn ~ 6500 2400
-NoConn ~ 2000 2000
-NoConn ~ 1600 1600
-NoConn ~ 1700 1600
-NoConn ~ 1800 1600
 Wire Wire Line
 	3200 1750 3200 1900
@@
 	9650 2000 9900 2000
 Wire Wire Line
-	1400 1250 1400 1600
-Wire Wire Line
 	5900 3400 5900 3750
 Wire Notes Line
@@
 	700  5050 4150 5050
 Wire Notes Line
-	4150 5050 4150 7650
-Wire Notes Line
-	4150 7650 700  7650
-Wire Notes Line
-	700  7650 700  5050
+	4150 5050 4150 6750
+Wire Notes Line
+	4150 6750 700  6750
+Wire Notes Line
+	700  6750 700  5050
 Wire Wire Line
 	7450 1250 9850 1250
@@
 Text Notes 700  5050 0    50   ~ 0
 Addressable Strip Connection
-$Comp
-L Connector:Conn_01x02_Male J4
-U 1 1 6096D0BC
+Wire Wire Line
+	1550 2550 1550 2500
+Wire Wire Line
+	1550 2350 1100 2350
+Wire Wire Line
+	1100 1250 1400 1250
+Wire Wire Line
+	1650 2550 1650 2500
+Wire Wire Line
+	1650 2350 2150 2350
+Wire Wire Line
+	2150 2350 2150 1900
+Wire Wire Line
+	1400 1250 2150 1250
+Connection ~ 2150 1250
+Wire Wire Line
+	2150 1250 2400 1250
+$Comp
+L Device:Fuse F1
+U 1 1 60A11576
+P 1100 1800
+F 0 "F1" H 1160 1846 50  0000 L CNN
+F 1 "Fuse" H 1160 1755 50  0000 L CNN
+F 2 "halibs:Fuse-PTF75_Stelvio" V 1030 1800 50  0001 C CNN
+F 3 "~" H 1100 1800 50  0001 C CNN
+	1    1100 1800
+	1    0    0    -1
+$EndComp
+Wire Wire Line
+	1100 1650 1100 1250
+Wire Wire Line
+	1100 2350 1100 1950
+$Comp
+L Connector:Conn_01x04_Male J1
+U 1 1 60A1F65F
 P 1550 2750
-F 0 "J4" V 1704 2562 50  0000 R CNN
-F 1 "Conn_01x02_Male" V 1613 2562 50  0000 R CNN
-F 2 "TerminalBlock:TerminalBlock_bornier-2_P5.08mm" H 1550 2750 50  0001 C CNN
+F 0 "J1" V 1704 2462 50  0000 R CNN
+F 1 "Conn_01x04_Male" V 1613 2462 50  0000 R CNN
+F 2 "TerminalBlock_Phoenix:TerminalBlock_Phoenix_MPT-0,5-4-2.54_1x04_P2.54mm_Horizontal" H 1550 2750 50  0001 C CNN
 F 3 "~" H 1550 2750 50  0001 C CNN
 	1    1550 2750
@@
 $EndComp
 Wire Wire Line
-	1550 2550 1550 2350
-Wire Wire Line
-	1550 2350 1100 2350
-Wire Wire Line
-	1100 2350 1100 1250
-Wire Wire Line
-	1100 1250 1400 1250
-Wire Wire Line
-	1650 2550 1650 2350
-Wire Wire Line
-	1650 2350 2150 2350
-Wire Wire Line
-	2150 2350 2150 1900
-Wire Wire Line
-	1400 1250 2150 1250
-Connection ~ 2150 1250
-Wire Wire Line
-	2150 1250 2400 1250
+	1450 2550 1450 2500
+Wire Wire Line
+	1450 2500 1550 2500
+Connection ~ 1550 2500
+Wire Wire Line
+	1550 2500 1550 2350
+Wire Wire Line
+	1750 2550 1750 2500
+Wire Wire Line
+	1750 2500 1650 2500
+Connection ~ 1650 2500
+Wire Wire Line
+	1650 2500 1650 2350
+Text Label 1200 2350 0    50   ~ 0
+SUPPLY
 $EndSCHEMATC

Commit message: Readme
Parts:
- C1, C2: value 100µF -> 100nF
Changed lines of the file:
@@
 Sheet 1 1
 Title "WS2812 Controller"
-Date "2021-05-12"
-Rev "0.3"
+Date "2021-06-10"
+Rev "0.4"
 Comp "haus-automatisierung.com"
 Comment1 "Matthias Kleine"
@@
 P 2150 1550
 F 0 "C1" H 2265 1596 50  0000 L CNN
-F 1 "100µF" H 2265 1505 50  0000 L CNN
+F 1 "100nF" H 2265 1505 50  0000 L CNN
 F 2 "Capacitor_SMD:C_0805_2012Metric_Pad1.15x1.40mm_HandSolder" H 2188 1400 50  0001 C CNN
 F 3 "~" H 2150 1550 50  0001 C CNN
@@
 P 3200 1600
 F 0 "C2" H 3315 1646 50  0000 L CNN
-F 1 "100µF" H 3315 1555 50  0000 L CNN
+F 1 "100nF" H 3315 1555 50  0000 L CNN
 F 2 "Capacitor_SMD:C_0805_2012Metric_Pad1.15x1.40mm_HandSolder" H 3238 1450 50  0001 C CNN
 F 3 "~" H 3200 1600 50  0001 C CNN

Commit message: v0.4
Parts:
- added U3: SN74AHCT125, halibs:SN74AHCT125D, symbol haus-automatisierung:SN74AHCT125
Connections:
- net +5V: now also U3.14 (VCC)
- net GND: now also J1.1 (Pin_1), J1.2 (Pin_2), U3.1 (1OE), U3.10 (3OE), U3.13 (4OE), U3.4 (2OE), U3.7 (GND); no longer J1.3 (Pin_3), J1.4 (Pin_4)
- net GPIO4: now also U3.2 (1A); no longer R6.2
- net SUPPLY: now also J1.3 (Pin_3), J1.4 (Pin_4); no longer J1.1 (Pin_1), J1.2 (Pin_2)
- new net DATA: R6.2, U3.3 (1Y)
- no-connect marks 12 -> 18
Other:
- note added: "Level Shifter"
- moved on the sheet: C3, J3, R6
Changed lines of the file:
@@
 Sheet 1 1
 Title "WS2812 Controller"
-Date "2021-06-21"
+Date "2021-09-29"
 Rev "0.4"
 Comp "haus-automatisierung.com"
@@
 Wire Wire Line
 	2150 1700 2150 1900
-Connection ~ 2150 1900
 Wire Wire Line
 	2150 1900 2700 1900
@@
 	700  600  10850 600
 Wire Notes Line
-	10850 600  10850 4650
-Wire Notes Line
-	10850 4650 700  4650
-Wire Notes Line
-	700  4650 700  600
+	10850 600  10850 4100
+Wire Notes Line
+	10850 4100 700  4100
+Wire Notes Line
+	700  4100 700  600
 Text GLabel 6600 1800 2    50   Input ~ 0
 TX
@@
 Wire Wire Line
 	6600 2100 6500 2100
-Text GLabel 2150 5800 0    50   Output ~ 0
-GPIO4
 $Comp
 L Connector_Generic:Conn_01x03 J3
 U 1 1 5DE1E3B4
-P 3500 5800
-F 0 "J3" H 3580 5842 50  0000 L CNN
-F 1 "Conn_01x03" H 3580 5751 50  0000 L CNN
-F 2 "TerminalBlock_Phoenix:TerminalBlock_Phoenix_MPT-0,5-3-2.54_1x03_P2.54mm_Horizontal" H 3500 5800 50  0001 C CNN
-F 3 "~" H 3500 5800 50  0001 C CNN
-	1    3500 5800
+P 3500 5400
+F 0 "J3" H 3580 5442 50  0000 L CNN
+F 1 "Conn_01x03" H 3580 5351 50  0000 L CNN
+F 2 "TerminalBlock_Phoenix:TerminalBlock_Phoenix_MPT-0,5-3-2.54_1x03_P2.54mm_Horizontal" H 3500 5400 50  0001 C CNN
+F 3 "~" H 3500 5400 50  0001 C CNN
+	1    3500 5400
 	1    0    0    -1
 $EndComp
@@
 L Device:R R6
 U 1 1 5DE21182
-P 2650 5800
-F 0 "R6" V 2443 5800 50  0000 C CNN
-F 1 "330Ω" V 2534 5800 50  0000 C CNN
-F 2 "Resistor_SMD:R_0805_2012Metric_Pad1.15x1.40mm_HandSolder" V 2580 5800 50  0001 C CNN
-F 3 "~" H 2650 5800 50  0001 C CNN
-	1    2650 5800
+P 2650 5400
+F 0 "R6" V 2443 5400 50  0000 C CNN
+F 1 "330Ω" V 2534 5400 50  0000 C CNN
+F 2 "Resistor_SMD:R_0805_2012Metric_Pad1.15x1.40mm_HandSolder" V 2580 5400 50  0001 C CNN
+F 3 "~" H 2650 5400 50  0001 C CNN
+	1    2650 5400
 	0    1    1    0
 $EndComp
 Wire Wire Line
-	2500 5800 2150 5800
-Wire Wire Line
-	2800 5800 3300 5800
+	2800 5400 3300 5400
 $Comp
 L power:+5V #PWR0101
 U 1 1 5DE276B5
-P 3150 5400
-F 0 "#PWR0101" H 3150 5250 50  0001 C CNN
-F 1 "+5V" H 3165 5573 50  0000 C CNN
-F 2 "" H 3150 5400 50  0001 C CNN
-F 3 "" H 3150 5400 50  0001 C CNN
-	1    3150 5400
-	1    0    0    -1
-$EndComp
-Wire Wire Line
-	3150 5400 3150 5700
-Wire Wire Line
-	3150 5700 3300 5700
+P 3150 5000
+F 0 "#PWR0101" H 3150 4850 50  0001 C CNN
+F 1 "+5V" H 3165 5173 50  0000 C CNN
+F 2 "" H 3150 5000 50  0001 C CNN
+F 3 "" H 3150 5000 50  0001 C CNN
+	1    3150 5000
+	1    0    0    -1
+$EndComp
+Wire Wire Line
+	3150 5000 3150 5300
+Wire Wire Line
+	3150 5300 3300 5300
 $Comp
 L power:GND #PWR0102
 U 1 1 5DE29666
-P 3150 6350
-F 0 "#PWR0102" H 3150 6100 50  0001 C CNN
-F 1 "GND" H 3155 6177 50  0000 C CNN
-F 2 "" H 3150 6350 50  0001 C CNN
-F 3 "" H 3150 6350 50  0001 C CNN
-	1    3150 6350
-	1    0    0    -1
-$EndComp
-Wire Wire Line
-	3150 6350 3150 5900
-Wire Wire Line
-	3150 5900 3300 5900
-Wire Wire Line
-	1300 5400 1300 5750
-Wire Wire Line
-	1300 6350 1300 6050
+P 3150 5950
+F 0 "#PWR0102" H 3150 5700 50  0001 C CNN
+F 1 "GND" H 3155 5777 50  0000 C CNN
+F 2 "" H 3150 5950 50  0001 C CNN
+F 3 "" H 3150 5950 50  0001 C CNN
+	1    3150 5950
+	1    0    0    -1
+$EndComp
+Wire Wire Line
+	3150 5950 3150 5500
+Wire Wire Line
+	3150 5500 3300 5500
+Wire Wire Line
+	1300 5000 1300 5350
+Wire Wire Line
+	1300 5950 1300 5650
 $Comp
 L power:GND #PWR06
 U 1 1 5DE0BC76
-P 1300 6350
-F 0 "#PWR06" H 1300 6100 50  0001 C CNN
-F 1 "GND" H 1305 6177 50  0000 C CNN
-F 2 "" H 1300 6350 50  0001 C CNN
-F 3 "" H 1300 6350 50  0001 C CNN
-	1    1300 6350
+P 1300 5950
+F 0 "#PWR06" H 1300 5700 50  0001 C CNN
+F 1 "GND" H 1305 5777 50  0000 C CNN
+F 2 "" H 1300 5950 50  0001 C CNN
+F 3 "" H 1300 5950 50  0001 C CNN
+	1    1300 5950
 	1    0    0    -1
 $EndComp
@@
 L power:+5V #PWR03
 U 1 1 5DE0B15D
-P 1300 5400
-F 0 "#PWR03" H 1300 5250 50  0001 C CNN
-F 1 "+5V" H 1315 5573 50  0000 C CNN
-F 2 "" H 1300 5400 50  0001 C CNN
-F 3 "" H 1300 5400 50  0001 C CNN
-	1    1300 5400
+P 1300 5000
+F 0 "#PWR03" H 1300 4850 50  0001 C CNN
+F 1 "+5V" H 1315 5173 50  0000 C CNN
+F 2 "" H 1300 5000 50  0001 C CNN
+F 3 "" H 1300 5000 50  0001 C CNN
+	1    1300 5000
 	1    0    0    -1
 $EndComp
@@
 L Device:CP C3
 U 1 1 5DE093FA
-P 1300 5900
-F 0 "C3" H 1418 5946 50  0000 L CNN
-F 1 "1000µF" H 1418 5855 50  0000 L CNN
-F 2 "Capacitor_THT:CP_Radial_D8.0mm_P3.80mm" H 1338 5750 50  0001 C CNN
-F 3 "~" H 1300 5900 50  0001 C CNN
-	1    1300 5900
-	1    0    0    -1
-$EndComp
-Wire Notes Line
-	700  5050 4150 5050
-Wire Notes Line
-	4150 5050 4150 6750
-Wire Notes Line
-	4150 6750 700  6750
-Wire Notes Line
-	700  6750 700  5050
+P 1300 5500
+F 0 "C3" H 1418 5546 50  0000 L CNN
+F 1 "1000µF" H 1418 5455 50  0000 L CNN
+F 2 "Capacitor_THT:CP_Radial_D8.0mm_P3.80mm" H 1338 5350 50  0001 C CNN
+F 3 "~" H 1300 5500 50  0001 C CNN
+	1    1300 5500
+	1    0    0    -1
+$EndComp
+Wire Notes Line
+	700  4650 4150 4650
+Wire Notes Line
+	4150 4650 4150 6350
+Wire Notes Line
+	4150 6350 700  6350
+Wire Notes Line
+	700  6350 700  4650
 Wire Wire Line
 	7450 1250 9850 1250
@@
 Wire Wire Line
 	4950 2050 4100 2050
-Text Notes 700  5050 0    50   ~ 0
+Text Notes 700  4650 0    50   ~ 0
 Addressable Strip Connection
 Wire Wire Line
-	1550 2550 1550 2500
-Wire Wire Line
-	1550 2350 1100 2350
-Wire Wire Line
 	1100 1250 1400 1250
-Wire Wire Line
-	1650 2550 1650 2500
-Wire Wire Line
-	1650 2350 2150 2350
-Wire Wire Line
-	2150 2350 2150 1900
 Wire Wire Line
 	1400 1250 2150 1250
@@
 Wire Wire Line
 	1100 1650 1100 1250
-Wire Wire Line
-	1100 2350 1100 1950
+Text Label 1100 2650 1    50   ~ 0
+SUPPLY
+$Comp
+L haus-automatisierung:SN74AHCT125 U3
+U 1 1 6154DBF8
+P 5850 5400
+F 0 "U3" H 6250 5300 50  0000 C CNN
+F 1 "SN74AHCT125" H 6200 5200 50  0000 C CNN
+F 2 "halibs:SN74AHCT125D" H 5850 5400 50  0001 C CNN
+F 3 "" H 5850 5400 50  0001 C CNN
+	1    5850 5400
+	1    0    0    -1
+$EndComp
+$Comp
+L power:+5V #PWR0104
+U 1 1 61550A59
+P 5850 5150
+F 0 "#PWR0104" H 5850 5000 50  0001 C CNN
+F 1 "+5V" H 5865 5323 50  0000 C CNN
+F 2 "" H 5850 5150 50  0001 C CNN
+F 3 "" H 5850 5150 50  0001 C CNN
+	1    5850 5150
+	1    0    0    -1
+$EndComp
+Wire Wire Line
+	5850 5150 5850 5600
+$Comp
+L power:GND #PWR0105
+U 1 1 61553AD9
+P 5850 7000
+F 0 "#PWR0105" H 5850 6750 50  0001 C CNN
+F 1 "GND" H 5855 6827 50  0000 C CNN
+F 2 "" H 5850 7000 50  0001 C CNN
+F 3 "" H 5850 7000 50  0001 C CNN
+	1    5850 7000
+	1    0    0    -1
+$EndComp
+Wire Wire Line
+	5850 7000 5850 6800
+Wire Wire Line
+	5450 5850 4600 5850
+Wire Wire Line
+	4600 5850 4600 6150
+NoConn ~ 6250 5950
+NoConn ~ 6250 6050
+NoConn ~ 6250 6250
+NoConn ~ 6250 6350
+NoConn ~ 5450 6250
+NoConn ~ 5450 6350
+Text GLabel 5100 6050 0    50   Input ~ 0
+DATA
+Wire Wire Line
+	5450 6050 5100 6050
+Text GLabel 2150 5400 0    50   Output ~ 0
+DATA
+Wire Wire Line
+	2150 5400 2500 5400
+Wire Notes Line
+	4350 4650 6800 4650
+Wire Notes Line
+	6800 4650 6800 7500
+Wire Notes Line
+	6800 7500 4350 7500
+Wire Notes Line
+	4350 7500 4350 4650
+Text Notes 4350 4650 0    50   ~ 0
+Level Shifter
+Wire Wire Line
+	5100 5950 5450 5950
+Text GLabel 5100 5950 0    50   Output ~ 0
+GPIO4
+Wire Wire Line
+	5450 6150 4600 6150
+Wire Wire Line
+	5850 6800 4600 6800
+Wire Wire Line
+	4600 6800 4600 6150
+Connection ~ 5850 6800
+Wire Wire Line
+	5850 6800 5850 6600
+Connection ~ 4600 6150
+Wire Wire Line
+	6250 5850 6650 5850
+Wire Wire Line
+	6650 5850 6650 6150
+Wire Wire Line
+	6650 6800 5850 6800
+Wire Wire Line
+	6250 6150 6650 6150
+Connection ~ 6650 6150
+Wire Wire Line
+	6650 6150 6650 6800
 $Comp
 L Connector:Conn_01x04_Male J1
 U 1 1 60A1F65F
-P 1550 2750
-F 0 "J1" V 1704 2462 50  0000 R CNN
-F 1 "Conn_01x04_Male" V 1613 2462 50  0000 R CNN
-F 2 "TerminalBlock_Phoenix:TerminalBlock_Phoenix_MPT-0,5-4-2.54_1x04_P2.54mm_Horizontal" H 1550 2750 50  0001 C CNN
-F 3 "~" H 1550 2750 50  0001 C CNN
-	1    1550 2750
-	0    -1   -1   0
-$EndComp
-Wire Wire Line
-	1450 2550 1450 2500
-Wire Wire Line
-	1450 2500 1550 2500
-Connection ~ 1550 2500
-Wire Wire Line
-	1550 2500 1550 2350
-Wire Wire Line
-	1750 2550 1750 2500
-Wire Wire Line
-	1750 2500 1650 2500
-Connection ~ 1650 2500
-Wire Wire Line
-	1650 2500 1650 2350
-Text Label 1200 2350 0    50   ~ 0
-SUPPLY
+P 1650 2550
+F 0 "J1" V 1450 2550 50  0000 R CNN
+F 1 "Conn_01x04_Male" V 1550 2850 50  0000 R CNN
+F 2 "TerminalBlock_Phoenix:TerminalBlock_Phoenix_MPT-0,5-4-2.54_1x04_P2.54mm_Horizontal" H 1650 2550 50  0001 C CNN
+F 3 "~" H 1650 2550 50  0001 C CNN
+	1    1650 2550
+	0    1    1    0
+$EndComp
+Wire Wire Line
+	1550 2750 1450 2750
+Wire Wire Line
+	1100 2750 1100 1950
+Connection ~ 1450 2750
+Wire Wire Line
+	1450 2750 1100 2750
+Wire Wire Line
+	1650 2750 1750 2750
+Wire Wire Line
+	2150 2750 2150 1900
+Connection ~ 1750 2750
+Wire Wire Line
+	1750 2750 2150 2750
+Connection ~ 2150 1900
 $EndSCHEMATC
